File: ExtendedBoard/ExtendedBoard.sch (KiCad schematic (older format))
At the start: 53 parts

Commit message: zaloha pcb
Parts:
- removed J?: rgbGNDs, symbol Connector:Conn_01x16_Male
- added J1: Ard 04, Connector_PinHeader_2.54mm:PinHeader_1x08_P2.54mm_Vertical, symbol Connector:Conn_01x08_Male
- added J10: PINOUT conn 2, Connector_PinHeader_2.54mm:PinHeader_1x20_P2.54mm_Vertical, symbol Connector:Conn_01x20_Male
- added J11: PINOUT IR, Connector_PinHeader_2.54mm:PinHeader_1x03_P2.54mm_Vertical, symbol Connector:Conn_01x03_Female
- added J12, J14, J15: GNDpair1, Connector_PinHeader_2.54mm:PinHeader_1x04_P2.54mm_Vertical, symbol Connector:Conn_01x04_Female
- added J13: GNDpair2, Connector_PinHeader_2.54mm:PinHeader_1x04_P2.54mm_Vertical, symbol Connector:Conn_01x04_Female
- added J16: PINOUT conn 1, Connector_PinHeader_2.54mm:PinHeader_1x20_P2.54mm_Vertical, symbol Connector:Conn_01x20_Male
- added J2: Ard 03, Connector_PinHeader_2.54mm:PinHeader_1x06_P2.54mm_Vertical, symbol Connector:Conn_01x06_Male
- added J21: INPUTS_Ard02_01, Connector_PinHeader_2.54mm:PinHeader_1x05_P2.54mm_Vertical, symbol Connector:Conn_01x05_Male
- added J22: 12VOutput, Connector_PinHeader_2.54mm:PinHeader_1x02_P2.54mm_Vertical, symbol Connector:Conn_01x02_Male
- added J23: INPUTS_Ard02, Connector_PinHeader_2.54mm:PinHeader_1x05_P2.54mm_Vertical, symbol Connector:Conn_01x05_Male
- added J24: DeanTInput_01, Connector_PinHeader_2.54mm:PinHeader_1x02_P2.54mm_Vertical, symbol Connector:Conn_01x02_Male
- added J3: Ard04_1, Connector_PinHeader_2.54mm:PinHeader_1x08_P2.54mm_Vertical, symbol Connector:Conn_01x08_Female
- added J4: Ard 03_1, Connector_PinHeader_2.54mm:PinHeader_1x06_P2.54mm_Vertical, symbol Connector:Conn_01x06_Female
- added J5: Ard 01, Connector_PinHeader_2.54mm:PinHeader_1x10_P2.54mm_Vertical, symbol Connector:Conn_01x10_Male
- added J6: Ard 02, Connector_PinHeader_2.54mm:PinHeader_1x08_P2.54mm_Vertical, symbol Connector:Conn_01x08_Male
- added J7: Ard 01_1, Connector_PinHeader_2.54mm:PinHeader_1x10_P2.54mm_Vertical, symbol Connector:Conn_01x10_Female
- added J8: Ard 02_1, Connector_PinHeader_2.54mm:PinHeader_1x08_P2.54mm_Vertical, symbol Connector:Conn_01x08_Female
- added J9: Inputs_PCA9685A, Connector_PinHeader_2.54mm:PinHeader_1x05_P2.54mm_Vertical, symbol Connector:Conn_01x05_Female
- C1, C10, C11, C12, C13, C14, C15, C16, C2, C3, C4, C5, C6, C7, C8, C9: renamed from C?; value C_Small -> 100n; footprint (none) -> Capacitor_THT:C_Disc_D4.3mm_W1.9mm_P5.00mm
- J17, J18, J19, J20: renamed from J?; footprint (none) -> Connector_PinHeader_2.54mm:PinHeader_1x04_P2.54mm_Vertical
- R1, R10, R11, R12, R13, R14, R15, R16, R2, R3, R4, R5, R6, R7, R8, R9: renamed from R?; footprint (none) -> Resistor_THT:R_Axial_DIN0207_L6.3mm_D2.5mm_P10.16mm_Horizontal
- gave numbers to parts that had none: 16
Connections:
- net labels added: 12V+, 3V3+, 5V+, A0, A1, A2, A3, A4, A5, AREF, D04, D05, D06, D07, D08, D09, D10, D14, D15, D16, DI0, DI1, DI10, DI11, DI12, DI13, DI2, DI3, DI4, DI5, DI6, DI7, DI8, DI9, IOREF, LED04, LED05, LED06, LED07, LED08, LED09, LED10, LED14, LED15, LED16, RESET, SCL1, SDA1, VIN, Vcc
- net labels removed: D21, D22, D23, D31, D32, D33, D41, D42, D43, D51, LED21, LED22, LED23, LED31, LED32, LED33, LED41, LED42, LED43, LED51
- wire segments 64 -> 96
Other:
- note removed: "1) IRR napájení + digital pin (viz 4. bod)"
- note removed: "2) displej, napájení + I2C (viz 4. bod)"
- note removed: "3) Supply 5V IN + pinout VCC a GND"
- note removed: "4) PLED pinout - obecně Arduino pinout"
- note removed: "4.1 2x D pro spínání zdroje + IRR, arduino VCC, PLEDS PWM pinout, současně 4 (do zálohy?)"
- note removed: "4.2 I2C pinout"
- note removed: "4.x Celkem 8 kabelů Do krabičky + VCC + GND = 10 (udělat víceřadé, např -> I2C)"
- moved on the sheet: J18, J19, J20
