File: ExtendedBoard/Verz 01/ExtendedBoardCopy.kicad_pcb (KiCad board)
At the start: 2 copper layers, 99.9 x 100 mm, 72 parts, among them J17 PWMpair1, J18 PWMpair2, J19 PWMpair3, J20 PWMpair4, J5 Ard 01, J6 Ard 02, J7 Ard 01_1, J8 Ard 02_1, Q1 TIP120, Q10 TIP120, Q11 TIP120, Q12 TIP120, Q13 TIP120, Q14 TIP120, Q15 TIP120, Q16 TIP120, Q2 TIP120, Q3 TIP120, Q4 TIP120, Q5 TIP120, Q6 TIP120, Q7 TIP120, Q8 TIP120, Q9 TIP120

Commit message: zaloha verze 1
Parts:
- removed +12V1: 12VOutput, Connector_PinHeader_2.54mm:PinHeader_1x02_P2.54mm_Vertical
- removed +5V1, +5V2: SUP ++, Connector_PinHeader_2.54mm:PinHeader_1x07_P2.54mm_Vertical
- removed 12V1: INPUTS_Ard02, Connector_PinHeader_2.54mm:PinHeader_1x05_P2.54mm_Vertical
- removed the DH2 at (176.5, 85.1)
- removed DeanT1: DeanTInput_01, Connector_PinHeader_2.54mm:PinHeader_1x02_P2.54mm_Vertical
- removed IR1: PINOUT IR, Connector_PinHeader_2.54mm:PinHeader_1x03_P2.54mm_Vertical
- removed J17: PWMpair1, Connector_PinHeader_2.54mm:PinHeader_1x04_P2.54mm_Vertical
- removed SUPPLYard1: SUPPLYard, Connector_PinHeader_2.54mm:PinHeader_2x02_P2.54mm_Vertical
- removed Vcc1: PINOUT ard Supply, Connector_PinHeader_2.54mm:PinHeader_1x03_P2.54mm_Vertical
- added +12V: 12VOutput, Connector_PinHeader_2.54mm:PinHeader_1x02_P2.54mm_Vertical, F.Cu at (176.5, 64.8)
- added 12V: INPUTS_Ard02, Connector_PinHeader_2.54mm:PinHeader_1x05_P2.54mm_Vertical, F.Cu at (184.2, 64.8)
- added 5V: SUP ++, Connector_PinHeader_2.54mm:PinHeader_1x07_P2.54mm_Vertical, F.Cu at (166.4, 153.7)
- added 5V: SUP ++, Connector_PinHeader_2.54mm:PinHeader_1x07_P2.54mm_Vertical, F.Cu at (166.4, 157.5)
- added DH2: MountingHole_4.3mm_M4, MountingHole:MountingHole_4.3mm_M4, F.Cu at (175.9, 142.9)
- added DH2: MountingHole_4.3mm_M4, MountingHole:MountingHole_4.3mm_M4, F.Cu at (177.8, 83.8)
- added DeanT: DeanTInput_01, Connector_PinHeader_2.54mm:PinHeader_1x02_P2.54mm_Vertical, F.Cu at (171.4, 157.5)
- added GND: PINOUT GNDS, Connector_PinHeader_2.54mm:PinHeader_1x07_P2.54mm_Vertical, F.Cu at (147.3, 157.5)
- added IR: PINOUT IR, Connector_PinHeader_2.54mm:PinHeader_1x03_P2.54mm_Vertical, F.Cu at (181.6, 154.9)
- added PWM3: PWMpair1, Connector_PinHeader_2.54mm:PinHeader_1x04_P2.54mm_Vertical, F.Cu at (109.2, 64.8)
- added SUPPLY ARD: SUPPLYard, Connector_PinHeader_2.54mm:PinHeader_2x02_P2.54mm_Vertical, F.Cu at (188.0, 151.1)
- added Vcc: PINOUT ard Supply, Connector_PinHeader_2.54mm:PinHeader_1x03_P2.54mm_Vertical, F.Cu at (171.4, 153.7)
- moved GND 3.81 mm to (171.4, 149.9)
- moved R16 0.63 mm to (177.8, 136.5)
- renumbered GND1 to GND, GND2 to GND, J8 to J7, J20 to PWM0, J19 to PWM1, J18 to PWM2, Supply1 to Supply, TR1 to TR
Routing:
- net 5V+: track 59.7 -> 53.3 mm
- net LED15: track 51.2 -> 48.2 mm
- net LED05: track 117.9 -> 115.6 mm
- net DI10: track 42.4 -> 43.7 mm
- net D16: track 82.1 -> 81.4 mm
- net Vcc: track 119.6 -> 120.1 mm
Other:
- board text added: "1"
- board text added: "12V"
- board text added: "16"
- board text added: "5V"
- board text added: "AREF"
- board text added: "D0"
- board text added: "D1"
- board text added: "D10"
- board text added: "D11"
- board text added: "GND"
- board text added: "HomeLeds V2.1"
- board text added: "SCL"
- board text added: "SDA"
- board text added: "Vcc"
- board text added: "|~D10"
- board text added: "|~D11"
- board text added: "|~D3"
- board text added: "|~D5"
- board text added: "|~D6"
- board text added: "|~D9"
- board text added: "~D12"
- board text added: "~D13"
- board text added: "~D2"
- board text added: "~D4"
- board text added: "~D7"
- board text added: "~D8"

Commit message: zaloha
Other:
- board text added: "JLCJLCJLCJLC"
Changed lines of the file:
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@@
   (general
     (thickness 1.6)
-    (drawings 89)
+    (drawings 90)
     (tracks 412)
     (zones 0)
@@
     (0 F.Cu signal)
     (31 B.Cu signal)
-    (32 B.Adhes user)
-    (33 F.Adhes user)
+    (32 B.Adhes user hide)
+    (33 F.Adhes user hide)
     (34 B.Paste user)
     (35 F.Paste user)
@@
     (38 B.Mask user)
     (39 F.Mask user)
-    (40 Dwgs.User user)
-    (41 Cmts.User user)
-    (42 Eco1.User user)
-    (43 Eco2.User user)
+    (40 Dwgs.User user hide)
+    (41 Cmts.User user hide)
+    (42 Eco1.User user hide)
+    (43 Eco2.User user hide)
     (44 Edge.Cuts user)
     (45 Margin user)
-    (46 B.CrtYd user)
-    (47 F.CrtYd user)
-    (48 B.Fab user)
-    (49 F.Fab user)
+    (46 B.CrtYd user hide)
+    (47 F.CrtYd user hide)
+    (48 B.Fab user hide)
+    (49 F.Fab user hide)
   )
   (setup
-    (last_trace_width 1)
+    (last_trace_width 0.25)
     (user_trace_width 0.4)
     (user_trace_width 0.6)
@@
       (effects (font (size 1 1) (thickness 0.15)))
     )
-    (fp_text user %R (at 0 7.62) (layer F.Fab)
-      (effects (font (size 1 1) (thickness 0.15)))
-    )
     (fp_line (start 1.8 -1.8) (end -1.8 -1.8) (layer F.CrtYd) (width 0.05))
     (fp_line (start 1.8 17.05) (end 1.8 -1.8) (layer F.CrtYd) (width 0.05))
@@
     (fp_line (start 1.27 -1.27) (end 1.27 16.51) (layer F.Fab) (width 0.1))
     (fp_line (start -0.635 -1.27) (end 1.27 -1.27) (layer F.Fab) (width 0.1))
+    (fp_text user %R (at 0 7.62) (layer F.Fab)
+      (effects (font (size 1 1) (thickness 0.15)))
+    )
     (pad 1 thru_hole rect (at 0 0 270) (size 1.7 1.7) (drill 1) (layers *.Cu *.Mask))
     (pad 2 thru_hole oval (at 0 2.54 270) (size 1.7 1.7) (drill 1) (layers *.Cu *.Mask))
@@
     )
   )
+  (gr_text JLCJLCJLCJLC (at 116.84 158.75) (layer F.SilkS)
+    (effects (font (size 1.5 1.5) (thickness 0.3)))
+  )
   (gr_text GND (at 132.08 159.325) (layer F.SilkS)
